File: Weslie_source_files/Weslie.kicad_pcb (KiCad board)
At the start: 2 copper layers, 34 parts, among them Q2 2N4401, Q3 MPF102

Commit message: Priemr entrega
Parts:
- added C1: 0.22U, Capacitor_THT:C_Disc_D10.0mm_W2.5mm_P5.00mm, F.Cu at (72.4, 86.3)
- added D2: LED_Small, LED_THT:LED_D3.0mm, F.Cu at (88.4, 101.6)
- added J1: in, Connector_Pin:Pin_D1.0mm_L10.0mm, F.Cu at (105.9, 100.3)
- added J2: out, Connector_Pin:Pin_D1.0mm_L10.0mm, F.Cu at (67.3, 101.3)
- added J3: 9V, Connector_Pin:Pin_D1.0mm_L10.0mm, F.Cu at (101.1, 91.4)
- added J4: gnd, Connector_Pin:Pin_D1.0mm_L10.0mm, F.Cu at (101.1, 95.5)
- added Q1: 2N4401, Package_TO_SOT_THT:TO-92_Wide, F.Cu at (74.7, 71.9)
- added Q4: 2N4401, Package_TO_SOT_THT:TO-92_Wide, F.Cu at (97.0, 88.9)
- added R17: 22K, Resistor_THT:R_Axial_DIN0204_L3.6mm_D1.6mm_P7.62mm_Horizontal, F.Cu at (99.1, 113.3)
- added SW1: 3PDT, Library:3PD, F.Cu at (87.3, 113.0)
- R2: footprint Resistor_THT:R_Axial_DIN0204_L3.6mm_D1.6mm_P5.08mm_Horizontal -> Resistor_THT:R_Axial_DIN0204_L3.6mm_D1.6mm_P7.62mm_Horizontal
- moved C4 85.4 mm to (71.1, 100.0), turned to 90 degrees
- moved C6 84.5 mm to (78.2, 98.0), turned to 90 degrees
- moved C8 81.4 mm to (84.8, 95.5)
- moved R3 70.0 mm to (75.4, 66.8), turned to 180 degrees
- moved R11 69.3 mm to (80.0, 68.6), turned to -90 degrees
- moved Q2 68.2 mm to (77.0, 81.9), turned to -90 degrees
- moved R5 67.4 mm to (84.7, 76.3), turned to 90 degrees
- moved R4 67.0 mm to (71.4, 77.5), turned to 90 degrees
- moved R1 66.5 mm to (82.2, 68.6), turned to -90 degrees
- moved C2 65.6 mm to (65.5, 77.4), turned to 90 degrees
- moved R7 64.5 mm to (68.6, 88.9), turned to 90 degrees
- moved Q3 63.3 mm to (81.9, 91.7)
- moved D1 61.7 mm to (87.4, 86.9), turned to 90 degrees
- moved R13 60.6 mm to (105.2, 68.1), turned to -90 degrees
- moved R2 59.3 mm to (65.5, 88.9), turned to 90 degrees
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Connections:
- R16 pad 2: unconnected-(R16-Pad2) -> /EFFECT
- R6 pad 1: unconnected-(R6-Pad1) -> Net-(R6-Pad1)
Routing:
- net Net-(D1-Pad1): track 0.00 -> 62.3 mm
- net +9V: track 0.00 -> 44.7 mm
- net Net-(RV1-Pad1): track 0.00 -> 43.0 mm, vias 0 -> 2
- net /DRY: track 0.00 -> 42.8 mm
- net Net-(Q3-Pad3): track 0.00 -> 33.6 mm
- net /EFFECT: track 0.00 -> 32.8 mm
- net Net-(C1-Pad2): track 0.00 -> 30.1 mm
- net Net-(Q2-Pad2): track 0.00 -> 30.0 mm
- net Net-(C10-Pad1): track 0.00 -> 29.9 mm
- net Net-(SW1-Pad4): track 0.00 -> 25.3 mm
- net Net-(R13-Pad1): track 0.00 -> 25.0 mm
- net Net-(C9-Pad1): track 0.00 -> 23.7 mm
- net Net-(R11-Pad1): track 0.00 -> 20.8 mm
- net Net-(R6-Pad1): track 0.00 -> 17.7 mm
- net Net-(C4-Pad2): track 0.00 -> 16.9 mm
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- added copper zone on B.Cu, net GND
- added copper zone on F.Cu, net GND
Other:
- board outline added: 52.3 x 86.9 mm
- board text added: "9VCC"
- board text added: "IN"
- board text added: "OUT"
