File: Weslie_source_files/Weslie.kicad_sch (KiCad schematic)
At the start: 5 parts

Commit message: Schematic
Parts:
- added C? (x7): C_Small, symbol Device:C_Small
- added C? (x2): C_Polarized, symbol Device:C_Polarized
- added D?: D_Zener, symbol Device:D_Zener
- added J?: AudioJack2_Ground, symbol Connector:AudioJack2_Ground
- added Q?: Q_NPN_ECB, symbol Device:Q_NPN_ECB
- added Q?: 2N4401, symbol Device:Q_NPN_ECB
- added R? (x15): R_US, symbol Device:R_US
- added RV? (x2): 500KLin, symbol Device:R_Potentiometer_US
- added RV? (x2): R_Potentiometer_US, symbol Device:R_Potentiometer_US
- added RV?: 5KlLin, symbol Device:R_Potentiometer_US
- Q?: value Q_NJFET_DSG -> MPF102
- RV?: value R_Potentiometer_US -> 1KLog
Connections:
- net at C?.1: now also R?.2
- net at C?.2: now also Q?.3 (B), C?.1, R?.1, R?.1
- net GND: now reaches RV?.1
- net GND: now also C?.2, D?.2 (A), Q?.1 (E), R?.1, RV?.1, RV?.1, RV?.2
- net at RV?.2: now also C?.1
- net at RV?.3: now also R?.1
- net at R?.1: now also J?.T
- net at Q?.1 (E): now also R?.2
- net at Q?.2 (C): now also Q?.3 (B), R?.1, R?.2
- net at Q?.1 (D): now also C?.1, C?.2
- net at Q?.2 (S): now also D?.1 (K), R?.1, RV?.2, RV?.3
- net at Q?.3 (G): now also R?.1, R?.2
- new net: RV?.1, RV?.2
- new net: C?.2, R?.1 (x2)
- new net: C?.1, Q?.1 (E), R?.2
- new net: C?.2, C?.2, R?.2
- new net: RV?.1, RV?.3
- new net: C?.1, R?.1, R?.2
- new net: R?.1, RV?.3
- new net: C?.1, C?.1, R?.2
- new net: C?.2, Q?.2 (C), R?.1, R?.2, R?.2
- new net: C?.1, RV?.2
- new net: C?.1, C?.2, R?.2
- new net: C?.2, Q?.3 (B), R?.1
- new net: R?.2, RV?.2
- new net +9V: Q?.2 (C), R?.2, R?.2, R?.2
Other:
- moved on the sheet: C?, Q?, R?, RV?

Commit message: .gitignore
Parts:
- C1: renamed from C?; value C_Small -> 0.22U
- C10: renamed from C?; value C_Small -> 0.1u; footprint (none) -> Capacitor_THT:C_Disc_D10.0mm_W2.5mm_P5.00mm
- C2, C3: renamed from C?; value C_Small -> 0.22U; footprint (none) -> Capacitor_THT:C_Disc_D10.0mm_W2.5mm_P5.00mm
- C4: renamed from C?; value C_Small -> 0.1uF; footprint (none) -> Capacitor_THT:C_Disc_D10.0mm_W2.5mm_P5.00mm
- C5: renamed from C?; value C_Small -> 0.22u; footprint (none) -> Capacitor_THT:C_Disc_D10.0mm_W2.5mm_P5.00mm
- C6: renamed from C?; value C_Polarized -> 0.1u; footprint (none) -> Capacitor_THT:CP_Radial_D5.0mm_P2.50mm
- C7, C8: renamed from C?; value C_Small -> 0.01u; footprint (none) -> Capacitor_THT:C_Disc_D10.0mm_W2.5mm_P5.00mm
- C9: renamed from C?; value C_Polarized -> 4u7; footprint (none) -> Capacitor_THT:CP_Radial_D5.0mm_P2.50mm
- D1: renamed from D?; value D_Zener -> 5v6; footprint (none) -> Diode_THT:D_A-405_P7.62mm_Horizontal
- Q2: renamed from Q?; value Q_NPN_ECB -> 2N4401; footprint (none) -> Package_TO_SOT_THT:TO-92_Wide
- Q3: renamed from Q?; footprint (none) -> Package_TO_SOT_THT:TO-92_Wide
- Q4: renamed from Q?; value Q_NPN_ECB -> 2N4401
- R1: renamed from R?; value R_US -> 82K; footprint (none) -> Resistor_THT:R_Axial_DIN0204_L3.6mm_D1.6mm_P7.62mm_Horizontal
- R10: renamed from R?; value R_US -> 22K; footprint (none) -> Resistor_THT:R_Axial_DIN0204_L3.6mm_D1.6mm_P7.62mm_Horizontal
- R11: renamed from R?; value R_US -> 680R; footprint (none) -> Resistor_THT:R_Axial_DIN0204_L3.6mm_D1.6mm_P7.62mm_Horizontal
- R12, R9: renamed from R?; value R_US -> 470K; footprint (none) -> Resistor_THT:R_Axial_DIN0204_L3.6mm_D1.6mm_P7.62mm_Horizontal
- R13: renamed from R?; value R_US -> 1K; footprint (none) -> Resistor_THT:R_Axial_DIN0204_L3.6mm_D1.6mm_P7.62mm_Horizontal
- R14, R16, R6, R8: renamed from R?; value R_US -> 33K; footprint (none) -> Resistor_THT:R_Axial_DIN0204_L3.6mm_D1.6mm_P7.62mm_Horizontal
- R15: renamed from R?; value R_US -> 470R; footprint (none) -> Resistor_THT:R_Axial_DIN0204_L3.6mm_D1.6mm_P7.62mm_Horizontal
- R2: renamed from R?; value R_US -> 68K; footprint (none) -> Resistor_THT:R_Axial_DIN0204_L3.6mm_D1.6mm_P5.08mm_Horizontal
- R3: renamed from R?; value R_US -> 15K; footprint (none) -> Resistor_THT:R_Axial_DIN0204_L3.6mm_D1.6mm_P7.62mm_Horizontal
- R4: renamed from R?; value R_US -> 3M9; footprint (none) -> Resistor_THT:R_Axial_DIN0204_L3.6mm_D1.6mm_P7.62mm_Horizontal
- R5: renamed from R?; value R_US -> 100K; footprint (none) -> Resistor_THT:R_Axial_DIN0204_L3.6mm_D1.6mm_P7.62mm_Horizontal
- R7: renamed from R?; value R_US -> 1M; footprint (none) -> Resistor_THT:R_Axial_DIN0204_L3.6mm_D1.6mm_P7.62mm_Horizontal
- RV1: renamed from RV?; value R_Potentiometer_US -> 1K; footprint (none) -> Potentiometer_THT:Potentiometer_ACP_CA9-V10_Vertical_Hole
- RVAccent1, RVSpeed1, RVVol1, RVWeight1: renamed from RV?; footprint (none) -> Potentiometer_THT:Potentiometer_Alps_RK09L_Single_Vertical
- RVTone1: renamed from RV?; value R_Potentiometer_US -> 1K Lin; footprint (none) -> Potentiometer_THT:Potentiometer_Alps_RK09L_Single_Vertical
- gave numbers to parts that had none: 2
Connections:
- net GND: now also RVSpeed1.1, RVSpeed1.2, RVWeight1.1
- net at RVSpeed1.3: now also R3.1
- net at RVWeight1.3: now also R5.1
- net at J1.T: no longer R6.1

Commit message: Priemr entrega
Parts:
- removed J1: AudioJack2_Ground, symbol Connector:AudioJack2_Ground
- added D2: LED_Small, LED_THT:LED_D3.0mm, symbol Device:LED_Small
- added J1: in, Connector_Pin:Pin_D1.0mm_L10.0mm, symbol Connector:Conn_01x01_Male
- added J2: out, Connector_Pin:Pin_D1.0mm_L10.0mm, symbol Connector:Conn_01x01_Male
- added J3: 9V, Connector_Pin:Pin_D1.0mm_L10.0mm, symbol Connector:Conn_01x01_Male
- added J4: gnd, Connector_Pin:Pin_D1.0mm_L10.0mm, symbol Connector:Conn_01x01_Male
- added R17: 22K, Resistor_THT:R_Axial_DIN0204_L3.6mm_D1.6mm_P7.62mm_Horizontal, symbol Device:R_US
- added SW1: 3PDT, Library:3PD, symbol 3PDT:3PDT
- C1: footprint (none) -> Capacitor_THT:C_Disc_D10.0mm_W2.5mm_P5.00mm
- Q1, Q4: footprint (none) -> Package_TO_SOT_THT:TO-92_Wide
- R2: footprint Resistor_THT:R_Axial_DIN0204_L3.6mm_D1.6mm_P5.08mm_Horizontal -> Resistor_THT:R_Axial_DIN0204_L3.6mm_D1.6mm_P7.62mm_Horizontal
Connections:
- net +9V: now also D2.2 (A), J3.1 (Pin_1)
- net GND: now also J4.1 (Pin_1), SW1.3 (A), SW1.8 (C)
- net EFFECT: now reaches R16.2
- net EFFECT: now also SW1.1 (A)
- net at R6.1: now also SW1.5 (B)
- new net: D2.1 (K), R17.2
- new net: R17.1, SW1.6 (B)
- new net: J2.1 (Pin_1), SW1.4 (B)
- new net DRY: J1.1 (Pin_1), SW1.2 (A), SW1.7 (C)
